File: tempcontroll/_saved_tempcontroll.sch (KiCad schematic (older format))
At the start: 59 parts, among them J1 REL1, J10 REL2B, J11 Conn_01x03, J12 AVR_SPI, J2 -5V, J3 +24V, J4 +5V, J5 GND, J6 +D, J7 -TS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

Commit message: Final pcb
Parts:
- R21, R22: value 1k -> 4k7
- gave numbers to parts that had none: 2
Changed lines of the file:
@@
 P 2700 2350
 F 0 "R21" V 2493 2350 50  0000 C CNN
-F 1 "1k" V 2584 2350 50  0000 C CNN
+F 1 "4k7" V 2584 2350 50  0000 C CNN
 F 2 "Resistors_SMD:R_0805" V 2630 2350 50  0001 C CNN
 F 3 "" H 2700 2350 50  0001 C CNN
@@
 P 2400 4200
 F 0 "R22" V 2300 4250 50  0000 R CNN
-F 1 "1k" V 2500 4250 50  0000 R CNN
+F 1 "4k7" V 2500 4250 50  0000 R CNN
 F 2 "Resistors_SMD:R_0805" V 2330 4200 50  0001 C CNN
 F 3 "" H 2400 4200 50  0001 C CNN
@@
 	3450 3200 3500 3200
 $Comp
-L device:Q_NPN_ECB Q?
+L device:Q_NPN_ECB Q5
 U 1 1 5A409982
 P 2250 2350
-F 0 "Q?" H 2100 2450 50  0000 L CNN
+F 0 "Q5" H 2100 2450 50  0000 L CNN
 F 1 "2SD667" H 1950 2200 50  0000 L CNN
 F 2 "TO_SOT_Packages_THT:TO-92_Molded_Narrow" H 2450 2450 50  0001 C CNN
@@
 	2150 2100 2150 2150
 $Comp
-L power:GND #PWR?
+L power:GND #PWR023
 U 1 1 5A412B11
 P 2150 2650
-F 0 "#PWR?" H 2150 2400 50  0001 C CNN
+F 0 "#PWR023" H 2150 2400 50  0001 C CNN
 F 1 "GND" H 2155 2477 50  0000 C CNN
 F 2 "" H 2150 2650 50  0001 C CNN
@@
 	2450 2350 2550 2350
 $Comp
-L device:Q_NPN_ECB Q?
+L device:Q_NPN_ECB Q4
 U 1 1 5A424860
 P 1900 4200
-F 0 "Q?" H 1750 4300 50  0000 L CNN
+F 0 "Q4" H 1750 4300 50  0000 L CNN
 F 1 "2SD667" H 1600 4050 50  0000 L CNN
 F 2 "TO_SOT_Packages_THT:TO-92_Molded_Narrow" H 2100 4300 50  0001 C CNN
@@
 	1800 3900 1800 4000
 $Comp
-L power:GND #PWR?
+L power:GND #PWR032
 U 1 1 5A42DD0E
 P 1800 4500
-F 0 "#PWR?" H 1800 4250 50  0001 C CNN
+F 0 "#PWR032" H 1800 4250 50  0001 C CNN
 F 1 "GND" H 1805 4327 50  0000 C CNN
 F 2 "" H 1800 4500 50  0001 C CNN
