File: tempcontroll/tempcontroll.kicad_pcb (KiCad board)
At the start: 2 copper layers, 80 x 80 mm, 27 parts, among them J1 AVR_SPI, J2 Conn_01x03, U1 ATMEGA8-16AU, U2 KL-4031-BSR, U3 OP07

Commit message: Start work
Parts:
- added C4: 100u, Capacitors_SMD:C_0805, B.Cu at (120.7, 71.1)
- added C5: 100u, Capacitors_SMD:C_0805, B.Cu at (133.6, 95.2)
- added C6: 100u, Capacitors_SMD:C_0805, B.Cu at (133.6, 97.8)
- added C7: 100u, Capacitors_SMD:C_0805, B.Cu at (109.8, 115.6)
- added C8: 100u, Capacitors_SMD:C_0805, B.Cu at (113.0, 71.1)
- added J10: REL2B, MY:PAD, F.Cu at (173.0, 65.0)
- added J11: Conn_01x03, Pin_Headers:Pin_Header_Straight_1x03_Pitch2.54mm, B.Cu at (154.9, 110.5)
- added J12: AVR_SPI, Pin_Headers:Pin_Header_Straight_2x03_Pitch2.54mm, B.Cu at (132.1, 85.1)
- added J3: +24V, MY:PAD, F.Cu at (117.0, 65.0)
- added J4: +5V, MY:PAD, F.Cu at (122.0, 65.0)
- added J5: GND, MY:PAD, F.Cu at (127.0, 65.0)
- added J6: +D, MY:PAD, F.Cu at (158.0, 65.0)
- added J7: -TS, MY:PAD, F.Cu at (153.0, 65.0)
- added J8: +TS, MY:PAD, F.Cu at (163.0, 65.0)
- added J9: REL2A, MY:PAD, F.Cu at (168.0, 65.0)
- added Q1: BC807, TO_SOT_Packages_SMD:SOT-23, B.Cu at (124.2, 44.8)
- added Q2: BC807, TO_SOT_Packages_SMD:SOT-23, B.Cu at (124.2, 49.2)
- added Q3: BC807, TO_SOT_Packages_SMD:SOT-23, B.Cu at (124.2, 53.7)
- added R18: 1k, Resistors_SMD:R_0805, B.Cu at (118.4, 45.7)
- added R19: 1k, Resistors_SMD:R_0805, B.Cu at (118.4, 50.2)
- added R20: 1k, Resistors_SMD:R_0805, B.Cu at (118.4, 54.6)
- J1: value AVR_SPI -> REL1; footprint Pin_Headers:Pin_Header_Straight_2x03_Pitch2.54mm -> MY:PAD; moved to F.Cu
- J2: value Conn_01x03 -> -5V; footprint Pin_Headers:Pin_Header_Straight_1x03_Pitch2.54mm -> MY:PAD
- R11: value 330 -> 10k
- R12: value 10k -> 330
- R2: value 10k -> 220
- R4: value 220 -> 10k
- U1: value ATMEGA8-16AU -> ATMEGA8-16PU; footprint Housings_QFP:LQFP-32_7x7mm_Pitch0.8mm -> Housings_DIP:DIP-28_W7.62mm; moved to F.Cu
- moved R4 50.2 mm to (150.8, 113.7), turned to 180 degrees
- moved J2 48.8 mm to (112.0, 65.0)
- moved J1 46.5 mm to (107.0, 65.0)
- moved R15 32.7 mm to (175.5, 92.5), turned to 90 degrees
- moved U3 32.5 mm to (165.2, 110.5), turned to 90 degrees
- moved U1 32.5 mm to (146.1, 110.5), turned to 180 degrees
- moved R2 30.2 mm to (144.8, 62.2), turned to 90 degrees
- moved D3 29.8 mm to (172.5, 98.0), turned to 90 degrees
- moved R13 25.1 mm to (170.0, 89.0), turned to 90 degrees
- moved R12 25.0 mm to (170.0, 92.6), turned to 90 degrees
- moved D4 20.6 mm to (165.4, 98.0), turned to 90 degrees
- moved R14 19.2 mm to (164.6, 85.5), turned to 90 degrees
- moved R10 19.1 mm to (138.4, 48.3), turned to 270 degrees
- moved R1 18.0 mm to (133.7, 92.7)
- moved R16 17.5 mm to (164.6, 89.0), turned to 90 degrees
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Connections:
- net Net-(R15-Pad1) renamed /TS
- J1 pad 1: /MISO -> Net-(J1-Pad1)
- J2 pad 1: GND -> -5V
- R11 pad 1: +5V -> Net-(C3-Pad1)
- R11 pad 2: Net-(D2-Pad2) -> Net-(R11-Pad2)
- R12 pad 1: Net-(C3-Pad1) -> +5V
- R12 pad 2: Net-(R12-Pad2) -> Net-(D2-Pad2)
- R2 pad 1: +5V -> Net-(R2-Pad1)
- R2 pad 2: /RES -> /G
- R3 pad 2: /G -> /DP
- R4 pad 1: Net-(R4-Pad1) -> +5V
- R4 pad 2: /DP -> /RES
- U1 pad 1: Net-(U1-Pad1) -> /RES
- U1 pad 10: Net-(U1-Pad10) -> Net-(R3-Pad1)
- U1 pad 12: Net-(R5-Pad2) -> Net-(U1-Pad12)
- U1 pad 13: Net-(R6-Pad2) -> /LED
- U1 pad 14: Net-(R7-Pad2) -> Net-(R5-Pad2)
- U1 pad 15: /MOSI -> Net-(R6-Pad2)
- U1 pad 16: /MISO -> Net-(R7-Pad2)
- U1 pad 17: /SCK -> /MOSI
- U1 pad 18: +5V -> /MISO
- U1 pad 19: Net-(U1-Pad19) -> /SCK
- U1 pad 2: Net-(U1-Pad2) -> /RX
- U1 pad 20: Net-(C1-Pad1) -> +5V
- U1 pad 21: GND -> Net-(C1-Pad1)
- U1 pad 22: Net-(U1-Pad22) -> GND
- U1 pad 23: Net-(R12-Pad2) -> Net-(R11-Pad2)
- U1 pad 3: GND -> /TX
- U1 pad 4: +5V -> Net-(U1-Pad4)
- U1 pad 5: GND -> Net-(U1-Pad5)
- U1 pad 6: +5V -> Net-(U1-Pad6)
- U1 pad 7: Net-(R3-Pad1) -> +5V
- U1 pad 8: Net-(R4-Pad1) -> GND
- U1 pad 9: /LED -> Net-(R2-Pad1)
Routing:
- net +5V: track 0.00 -> 188.4 mm
- net /D1: track 0.00 -> 90.5 mm
- net /D2: track 0.00 -> 84.3 mm
- net /D3: track 0.00 -> 79.4 mm
- net GND: track 0.00 -> 63.7 mm
- net /SCK: track 0.00 -> 59.5 mm
- net Net-(R5-Pad2): track 0.00 -> 46.5 mm
- net /RES: track 0.00 -> 46.5 mm
- net Net-(R3-Pad1): track 0.00 -> 38.6 mm
- net Net-(R6-Pad2): track 0.00 -> 35.2 mm
- net /MISO: track 0.00 -> 32.5 mm
- net /MOSI: track 0.00 -> 32.0 mm
- net Net-(R2-Pad1): track 0.00 -> 29.1 mm
- net Net-(C1-Pad1): track 0.00 -> 22.8 mm
- net Net-(Q1-Pad3): track 0.00 -> 21.2 mm
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Other:
- net class Default: trace_width 0.25 -> 0.3556; via_dia 0.8 -> 2
- net class Power added: clearance 0.2, trace_width 0.4, via_dia 2, via_drill 0.4

Commit message: Job with pcb
Parts:
- moved R11 53.2 mm to (139.7, 115.2), turned to 90 degrees
- moved R15 24.1 mm to (165.1, 70.8), turned to 270 degrees
- moved U3 23.0 mm to (167.6, 87.6), turned to 270 degrees
- moved R17 21.9 mm to (162.6, 70.8), turned to 270 degrees
- moved D3 21.7 mm to (165.2, 77.5), turned to 0 degrees
- moved R12 20.2 mm to (149.9, 94.3)
- moved R14 17.7 mm to (161.6, 102.9), turned to 0 degrees
- moved R16 16.7 mm to (161.6, 105.4), turned to 180 degrees
- moved D4 15.4 mm to (165.2, 82.5), turned to 180 degrees
- moved R13 14.1 mm to (161.6, 100.3), turned to 0 degrees
- moved C8 2.81 mm to (115.8, 71.1)
- moved R7 2.54 mm to (139.7, 62.2)
Routing:
- net +5V: track 188.4 -> 343.7 mm, vias 0 -> 2
- net GND: track 63.7 -> 208.1 mm, vias 0 -> 2
- net -5V: track 6.13 -> 72.8 mm, vias 0 -> 2
- net Net-(D2-Pad2): track 0.00 -> 57.2 mm
- net /LED: track 0.00 -> 43.6 mm
- net Net-(C3-Pad1): track 0.00 -> 37.2 mm
- net Net-(D3-Pad2): track 0.00 -> 36.8 mm
- net Net-(R11-Pad2): track 0.00 -> 17.7 mm
- net Net-(D3-Pad1): track 0.00 -> 16.1 mm
- net Net-(R13-Pad1): track 0.00 -> 10.2 mm
- net /TS: track 0.00 -> 7.57 mm
- net /MOSI: track 32.0 -> 31.1 mm
- net Net-(R5-Pad2): track 46.5 -> 47.3 mm

Commit message: Finish work with pcb
Parts:
- moved C7 44.3 mm to (150.9, 99.1), turned to 180 degrees
Routing:
- net GND: track 208.1 -> 211.6 mm
- net Net-(R5-Pad2): track 47.3 -> 48.4 mm
- net +5V: track 343.7 -> 344.5 mm
Changed lines of the file:
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@@
     (thickness 1.6)
     (drawings 6)
-    (tracks 355)
+    (tracks 358)
     (zones 0)
     (modules 48)
@@
   )
   (module Capacitors_SMD:C_0805 (layer B.Cu)
-    (at 109.778952 115.6095)
+    (at 150.86 99.06 180)
     (descr "Capacitor SMD 0805, reflow soldering, AVX (see smccp.pdf)")
     (tags "capacitor 0805")
     (attr smd)
-    (fp_text reference C7 (at 0 1.5) (layer B.SilkS)
-      (effects (font (size 1 1) (thickness 0.15)) (justify mirror))
-    )
-    (fp_text value 100u (at 0 -1.75) (layer B.Fab)
-      (effects (font (size 1 1) (thickness 0.15)) (justify mirror))
-    )
-    (fp_text user %R (at 0 1.5) (layer B.Fab)
+    (fp_text reference C7 (at 0 1.5 180) (layer B.SilkS)
+      (effects (font (size 1 1) (thickness 0.15)) (justify mirror))
+    )
+    (fp_text value 100u (at 0 -1.75 180) (layer B.Fab)
+      (effects (font (size 1 1) (thickness 0.15)) (justify mirror))
+    )
+    (fp_text user %R (at 0 1.5 180) (layer B.Fab)
       (effects (font (size 1 1) (thickness 0.15)) (justify mirror))
     )
@@
     (fp_line (start 1.75 -0.87) (end 1.75 0.88) (layer B.CrtYd) (width 0.05))
     (fp_line (start 1.75 -0.87) (end -1.75 -0.87) (layer B.CrtYd) (width 0.05))
-    (pad 1 smd rect (at -1 0) (size 1 1.25) (layers B.Cu B.Paste B.Mask)
+    (pad 1 smd rect (at -1 0 180) (size 1 1.25) (layers B.Cu B.Paste B.Mask)
       (net 1 GND))
-    (pad 2 smd rect (at 1 0) (size 1 1.25) (layers B.Cu B.Paste B.Mask)
+    (pad 2 smd rect (at 1 0 180) (size 1 1.25) (layers B.Cu B.Paste B.Mask)
       (net 5 +5V))
     (model Capacitors_SMD.3dshapes/C_0805.wrl
@@
   (gr_line (start 100 40) (end 180 40) (layer Edge.Cuts) (width 0.2))
   (gr_line (start 100 120) (end 100 40) (layer Edge.Cuts) (width 0.2))
+  (segment (start 151.003 94.234) (end 155.067 98.298) (width 0.3556) (layer B.Cu) (net 1))
+  (segment (start 155.067 98.298) (end 157.099 100.33) (width 0.3556) (layer B.Cu) (net 1))
+  (segment (start 151.86 99.06) (end 154.305 99.06) (width 0.35) (layer B.Cu) (net 1))
+  (segment (start 154.305 99.06) (end 155.067 98.298) (width 0.35) (layer B.Cu) (net 1))
   (segment (start 141.478 86.995) (end 143.256 88.773) (width 0.3556) (layer B.Cu) (net 1))
   (segment (start 136.779 73.025) (end 136.779 77.978) (width 0.3556) (layer B.Cu) (net 1))
@@
   (segment (start 157.099 100.33) (end 157.099 110.49) (width 0.3556) (layer B.Cu) (net 1))
   (segment (start 147.574 94.234) (end 151.003 94.234) (width 0.3556) (layer B.Cu) (net 1))
-  (segment (start 151.003 94.234) (end 157.099 100.33) (width 0.3556) (layer B.Cu) (net 1))
   (segment (start 157.099 110.49) (end 161.29 110.49) (width 0.3556) (layer B.Cu) (net 1))
   (segment (start 154.94 110.49) (end 157.099 110.49) (width 0.3556) (layer B.Cu) (net 1))
@@
   (segment (start 129.54 85.09) (end 132.08 87.63) (width 0.4) (layer B.Cu) (net 4))
   (segment (start 132.08 87.63) (end 138.43 87.63) (width 0.4) (layer B.Cu) (net 4))
+  (segment (start 155.956 109.22) (end 156.41639 108.75961) (width 0.3556) (layer B.Cu) (net 5))
+  (segment (start 150.876 109.22) (end 155.956 109.22) (width 0.3556) (layer B.Cu) (net 5))
+  (segment (start 150.876 113.665) (end 150.876 109.22) (width 0.3556) (layer B.Cu) (net 5))
+  (segment (start 151.76 113.665) (end 150.876 113.665) (width 0.3556) (layer B.Cu) (net 5))
+  (segment (start 156.41639 103.07639) (end 154.94 101.6) (width 0.3556) (layer B.Cu) (net 5))
+  (segment (start 156.41639 108.75961) (end 156.41639 103.07639) (width 0.3556) (layer B.Cu) (net 5))
+  (segment (start 151.13 101.6) (end 154.94 101.6) (width 0.35) (layer B.Cu) (net 5))
+  (segment (start 149.86 100.33) (end 151.13 101.6) (width 0.35) (layer B.Cu) (net 5))
+  (segment (start 149.86 99.06) (end 149.86 100.33) (width 0.35) (layer B.Cu) (net 5))
+  (segment (start 149.86 96.52) (end 149.86 99.06) (width 0.35) (layer B.Cu) (net 5))
+  (segment (start 124.587 86.106) (end 128.651 90.17) (width 0.3556) (layer B.Cu) (net 5))
+  (segment (start 124.587 83.947) (end 124.587 86.106) (width 0.3556) (layer B.Cu) (net 5))
+  (segment (start 128.651 90.17) (end 132.715 90.17) (width 0.3556) (layer B.Cu) (net 5))
+  (segment (start 121.65 81.01) (end 124.587 83.947) (width 0.3556) (layer B.Cu) (net 5))
+  (segment (start 121.65 75.946) (end 121.65 81.01) (width 0.3556) (layer B.Cu) (net 5))
   (segment (start 149.86 96.52) (end 149.86 95.25) (width 0.35) (layer B.Cu) (net 5))
-  (segment (start 151.76 113.665) (end 151.0544 113.665) (width 0.3556) (layer B.Cu) (net 5))
-  (segment (start 151.0544 113.665) (end 151.0544 111.6844) (width 0.3556) (layer B.Cu) (net 5))
-  (segment (start 153.289 109.093) (end 153.458199 109.262199) (width 0.3556) (layer B.Cu) (net 5))
-  (segment (start 156.41639 108.75961) (end 156.41639 103.07639) (width 0.3556) (layer B.Cu) (net 5))
-  (segment (start 156.41639 103.07639) (end 151.003 97.663) (width 0.3556) (layer B.Cu) (net 5))
-  (segment (start 150.876 109.093) (end 153.289 109.093) (width 0.3556) (layer B.Cu) (net 5))
-  (segment (start 151.0544 111.6844) (end 150.876 111.506) (width 0.3556) (layer B.Cu) (net 5))
-  (segment (start 153.458199 109.262199) (end 155.913801 109.262199) (width 0.3556) (layer B.Cu) (net 5))
-  (segment (start 155.913801 109.262199) (end 156.41639 108.75961) (width 0.3556) (layer B.Cu) (net 5))
-  (segment (start 150.876 111.506) (end 150.876 109.093) (width 0.3556) (layer B.Cu) (net 5))
-  (segment (start 151.003 97.663) (end 149.86 96.52) (width 0.35) (layer B.Cu) (net 5))
   (segment (start 132.08 75.946) (end 132.08 77.360213) (width 0.3556) (layer B.Cu) (net 5))
   (segment (start 132.08 77.360213) (end 132.08 82.55) (width 0.3556) (layer B.Cu) (net 5))
   (via (at 132.08 75.946) (size 2) (drill 0.4) (layers F.Cu B.Cu) (net 5))
   (segment (start 121.65 75.946) (end 132.08 75.946) (width 0.3556) (layer F.Cu) (net 5))
-  (segment (start 121.65 75.946) (end 121.65 81.01) (width 0.3556) (layer B.Cu) (net 5))
   (segment (start 121.65 71.12) (end 121.65 75.946) (width 0.3556) (layer B.Cu) (net 5))
   (via (at 121.65 75.946) (size 2) (drill 0.4) (layers F.Cu B.Cu) (net 5))
@@
   (segment (start 165.1 95.25) (end 165.1 109.22) (width 0.3556) (layer B.Cu) (net 5))
   (segment (start 134.747 116.84) (end 134.747 115.316) (width 0.3556) (layer B.Cu) (net 5))
-  (segment (start 126.365 90.17) (end 132.715 90.17) (width 0.3556) (layer B.Cu) (net 5))
   (segment (start 132.715 90.17) (end 133.487 90.17) (width 0.3556) (layer B.Cu) (net 5))
   (segment (start 132.72 90.937) (end 132.72 90.175) (width 0.3556) (layer B.Cu) (net 5))
   (segment (start 132.72 90.175) (end 132.715 90.17) (width 0.3556) (layer B.Cu) (net 5))
-  (segment (start 124.587 88.392) (end 126.365 90.17) (width 0.3556) (layer B.Cu) (net 5))
-  (segment (start 124.587 83.947) (end 124.587 88.392) (width 0.3556) (layer B.Cu) (net 5))
-  (segment (start 121.65 81.01) (end 124.587 83.947) (width 0.3556) (layer B.Cu) (net 5))
   (segment (start 146.05 95.25) (end 147.18137 95.25) (width 0.3556) (layer B.Cu) (net 5))
   (segment (start 147.18137 95.25) (end 149.86 95.25) (width 0.3556) (layer B.Cu) (net 5))
@@
   (segment (start 144.018 85.598) (end 146.05 87.63) (width 0.35) (layer B.Cu) (net 20))
   (segment (start 148.59 53.34) (end 149.733 53.34) (width 0.35) (layer B.Cu) (net 20))
+  (segment (start 137.2824 51.562) (end 139.954 51.562) (width 0.35) (layer B.Cu) (net 21))
+  (segment (start 139.954 51.562) (end 140.081 51.435) (width 0.35) (layer B.Cu) (net 21))
+  (segment (start 135.89 51.562) (end 137.2824 51.562) (width 0.35) (layer B.Cu) (net 21))
+  (segment (start 135.89 49.9156) (end 135.89 51.562) (width 0.35) (layer B.Cu) (net 21))
   (segment (start 135.89 49.21) (end 135.89 49.9156) (width 0.3556) (layer B.Cu) (net 21))
-  (segment (start 135.89 49.9156) (end 137.4094 51.435) (width 0.3556) (layer B.Cu) (net 21))
-  (segment (start 137.4094 51.435) (end 139.115 51.435) (width 0.3556) (layer B.Cu) (net 21))
-  (segment (start 139.115 51.435) (end 140.081 51.435) (width 0.35) (layer B.Cu) (net 21))
   (segment (start 140.081 51.435) (end 143.256 48.26) (width 0.35) (layer B.Cu) (net 21))
   (segment (start 143.256 48.26) (end 147.828 48.26) (width 0.35) (layer B.Cu) (net 21))
@@
   (segment (start 128.458 44.77) (end 132.08 41.148) (width 0.4) (layer B.Cu) (net 50))
   (segment (start 125.19 44.77) (end 128.458 44.77) (width 0.4) (layer B.Cu) (net 50))
-  (segment (start 126.426 49.215) (end 127.508 48.133) (width 0.4) (layer B.Cu) (net 51))
-  (segment (start 127.508 48.133) (end 127.508 46.863) (width 0.4) (layer B.Cu) (net 51))
-  (segment (start 127.508 46.863) (end 132.334 42.037) (width 0.4) (layer B.Cu) (net 51))
+  (segment (start 131.445 42.926) (end 132.334 42.037) (width 0.4) (layer B.Cu) (net 51))
   (segment (start 125.19 49.215) (end 126.426 49.215) (width 0.4) (layer B.Cu) (net 51))
+  (segment (start 131.445 44.196) (end 131.445 42.926) (width 0.4) (layer B.Cu) (net 51))
+  (segment (start 126.426 49.215) (end 131.445 44.196) (width 0.4) (layer B.Cu) (net 51))
   (segment (start 132.334 42.037) (end 139.492 42.037) (width 0.4) (layer B.Cu) (net 51))
   (segment (start 139.492 42.037) (end 141.27 43.815) (width 0.4) (layer B.Cu) (net 51))

Commit message: Start coding 2
Routing:
- net /D3: track 79.4 -> 86.9 mm
- net /D2: track 84.3 -> 91.7 mm
- net /D1: track 90.5 -> 96.6 mm
- net +5V: track 344.5 -> 349.6 mm
Changed lines of the file:
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@@
-(kicad_pcb (version 20171130) (host pcbnew no-vcs-found-f4f0c09~61~ubuntu17.04.1)
+(kicad_pcb (version 20171130) (host pcbnew no-vcs-found-320fa71~61~ubuntu17.10.1)
   (general
     (thickness 1.6)
     (drawings 6)
-    (tracks 358)
+    (tracks 362)
     (zones 0)
     (modules 48)
@@
   )
   (setup
-    (last_trace_width 0.35)
+    (last_trace_width 0.3556)
     (user_trace_width 0.2)
     (user_trace_width 0.25)
@@
   (segment (start 129.54 85.09) (end 132.08 87.63) (width 0.4) (layer B.Cu) (net 4))
   (segment (start 132.08 87.63) (end 138.43 87.63) (width 0.4) (layer B.Cu) (net 4))
+  (segment (start 101.473 70.104) (end 109.982 78.613) (width 0.35) (layer B.Cu) (net 5))
+  (segment (start 101.473 58.293) (end 101.473 70.104) (width 0.35) (layer B.Cu) (net 5))
+  (segment (start 115.951 43.815) (end 101.473 58.293) (width 0.35) (layer B.Cu) (net 5))
+  (segment (start 123.19 43.82) (end 122.39 43.82) (width 0.35) (layer B.Cu) (net 5))
+  (segment (start 122.385 43.815) (end 115.951 43.815) (width 0.35) (layer B.Cu) (net 5))
+  (segment (start 109.982 78.613) (end 109.982 99.314) (width 0.35) (layer B.Cu) (net 5))
+  (segment (start 122.39 43.82) (end 122.385 43.815) (width 0.35) (layer B.Cu) (net 5))
+  (segment (start 109.982 99.314) (end 118.618 107.95) (width 0.35) (layer B.Cu) (net 5))
+  (segment (start 118.618 107.95) (end 127.381 107.95) (width 0.35) (layer B.Cu) (net 5))
+  (segment (start 127.381 107.95) (end 134.747 115.316) (width 0.35) (layer B.Cu) (net 5))
   (segment (start 155.956 109.22) (end 156.41639 108.75961) (width 0.3556) (layer B.Cu) (net 5))
   (segment (start 150.876 109.22) (end 155.956 109.22) (width 0.3556) (layer B.Cu) (net 5))
@@
   (segment (start 141.478 109.474) (end 141.478 115.189) (width 0.35) (layer B.Cu) (net 5))
   (segment (start 141.478 115.189) (end 141.605 115.316) (width 0.35) (layer B.Cu) (net 5))
-  (segment (start 118.364 98.933) (end 134.747 115.316) (width 0.35) (layer B.Cu) (net 5))
-  (segment (start 118.364 86.995) (end 118.364 98.933) (width 0.35) (layer B.Cu) (net 5))
-  (segment (start 101.473 70.104) (end 118.364 86.995) (width 0.35) (layer B.Cu) (net 5))
-  (segment (start 101.473 58.293) (end 101.473 70.104) (width 0.35) (layer B.Cu) (net 5))
-  (segment (start 115.951 43.815) (end 101.473 58.293) (width 0.35) (layer B.Cu) (net 5))
-  (segment (start 122.385 43.815) (end 115.951 43.815) (width 0.35) (layer B.Cu) (net 5))
-  (segment (start 123.19 43.82) (end 122.39 43.82) (width 0.35) (layer B.Cu) (net 5))
-  (segment (start 122.39 43.82) (end 122.385 43.815) (width 0.35) (layer B.Cu) (net 5))
   (segment (start 151.765 115.316) (end 151.76 115.311) (width 0.35) (layer B.Cu) (net 5))
   (segment (start 141.478 91.567) (end 141.478 109.474) (width 0.35) (layer B.Cu) (net 5))
@@
   (segment (start 149.352 76.708) (end 149.352 64.643) (width 0.3556) (layer B.Cu) (net 27))
   (segment (start 146.05 80.01) (end 149.352 76.708) (width 0.3556) (layer B.Cu) (net 27))
-  (segment (start 102.235 69.723) (end 119.126 86.614) (width 0.4) (layer B.Cu) (net 28))
-  (segment (start 119.126 86.614) (end 119.126 96.647) (width 0.4) (layer B.Cu) (net 28))
-  (segment (start 102.235 58.801) (end 102.235 69.723) (width 0.4) (layer B.Cu) (net 28))
-  (segment (start 115.316 45.72) (end 102.235 58.801) (width 0.4) (layer B.Cu) (net 28))
-  (segment (start 117.48 45.72) (end 115.316 45.72) (width 0.4) (layer B.Cu) (net 28))
-  (segment (start 119.126 96.647) (end 132.969 110.49) (width 0.4) (layer B.Cu) (net 28))
-  (segment (start 132.969 110.49) (end 137.29863 110.49) (width 0.4) (layer B.Cu) (net 28))
-  (segment (start 137.29863 110.49) (end 138.43 110.49) (width 0.4) (layer B.Cu) (net 28))
-  (segment (start 119.888 96.266) (end 131.572 107.95) (width 0.4) (layer B.Cu) (net 29))
-  (segment (start 102.997 61.468) (end 102.997 69.469) (width 0.4) (layer B.Cu) (net 29))
-  (segment (start 119.888 86.36) (end 119.888 96.266) (width 0.4) (layer B.Cu) (net 29))
-  (segment (start 102.997 69.469) (end 119.888 86.36) (width 0.4) (layer B.Cu) (net 29))
-  (segment (start 114.3 50.165) (end 102.997 61.468) (width 0.4) (layer B.Cu) (net 29))
-  (segment (start 117.48 50.165) (end 114.3 50.165) (width 0.4) (layer B.Cu) (net 29))
-  (segment (start 131.572 107.95) (end 137.29863 107.95) (width 0.4) (layer B.Cu) (net 29))
-  (segment (start 137.29863 107.95) (end 138.43 107.95) (width 0.4) (layer B.Cu) (net 29))
-  (segment (start 120.777 95.885) (end 130.302 105.41) (width 0.4) (layer B.Cu) (net 30))
-  (segment (start 120.777 86.233) (end 120.777 95.885) (width 0.4) (layer B.Cu) (net 30))
-  (segment (start 103.759 61.849) (end 103.759 69.215) (width 0.4) (layer B.Cu) (net 30))
-  (segment (start 117.48 54.61) (end 110.998 54.61) (width 0.4) (layer B.Cu) (net 30))
-  (segment (start 103.759 69.215) (end 120.777 86.233) (width 0.4) (layer B.Cu) (net 30))
-  (segment (start 110.998 54.61) (end 103.759 61.849) (width 0.4) (layer B.Cu) (net 30))
-  (segment (start 130.302 105.41) (end 138.43 105.41) (width 0.4) (layer B.Cu) (net 30))
+  (segment (start 110.744 98.933) (end 118.872 107.061) (width 0.4) (layer B.Cu) (net 28))
+  (segment (start 102.235 69.723) (end 110.744 78.232) (width 0.4) (layer B.Cu) (net 28))
+  (segment (start 102.235 59.055) (end 102.235 69.723) (width 0.4) (layer B.Cu) (net 28))
+  (segment (start 118.872 107.061) (end 135.001 107.061) (width 0.4) (layer B.Cu) (net 28))
+  (segment (start 117.48 45.72) (end 115.57 45.72) (width 0.4) (layer B.Cu) (net 28))
+  (segment (start 110.744 78.232) (end 110.744 98.933) (width 0.4) (layer B.Cu) (net 28))
+  (segment (start 115.57 45.72) (end 102.235 59.055) (width 0.4) (layer B.Cu) (net 28))
+  (segment (start 135.001 107.061) (end 137.630001 109.690001) (width 0.4) (layer B.Cu) (net 28))
+  (segment (start 137.630001 109.690001) (end 138.43 110.49) (width 0.4) (layer B.Cu) (net 28))
+  (segment (start 111.413989 98.459989) (end 119.126 106.172) (width 0.4) (layer B.Cu) (net 29))
+  (segment (start 102.997 69.469) (end 111.413989 77.885989) (width 0.4) (layer B.Cu) (net 29))
+  (segment (start 102.997 59.563) (end 102.997 69.469) (width 0.4) (layer B.Cu) (net 29))
+  (segment (start 111.413989 77.885989) (end 111.413989 98.459989) (width 0.4) (layer B.Cu) (net 29))
+  (segment (start 117.48 50.165) (end 112.395 50.165) (width 0.4) (layer B.Cu) (net 29))
+  (segment (start 112.395 50.165) (end 102.997 59.563) (width 0.4) (layer B.Cu) (net 29))
+  (segment (start 119.126 106.172) (end 136.652 106.172) (width 0.4) (layer B.Cu) (net 29))
+  (segment (start 136.652 106.172) (end 137.630001 107.150001) (width 0.4) (layer B.Cu) (net 29))
+  (segment (start 137.630001 107.150001) (end 138.43 107.95) (width 0.4) (layer B.Cu) (net 29))
+  (segment (start 112.141 98.171) (end 119.38 105.41) (width 0.4) (layer B.Cu) (net 30))
+  (segment (start 103.759 69.215) (end 112.141 77.597) (width 0.4) (layer B.Cu) (net 30))
+  (segment (start 103.759 59.944) (end 103.759 69.215) (width 0.4) (layer B.Cu) (net 30))
+  (segment (start 117.48 54.61) (end 109.093 54.61) (width 0.4) (layer B.Cu) (net 30))
+  (segment (start 112.141 77.597) (end 112.141 98.171) (width 0.4) (layer B.Cu) (net 30))
+  (segment (start 109.093 54.61) (end 103.759 59.944) (width 0.4) (layer B.Cu) (net 30))
+  (segment (start 119.38 105.41) (end 138.43 105.41) (width 0.4) (layer B.Cu) (net 30))
   (segment (start 162.56 71.75) (end 162.56 73.787) (width 0.3556) (layer B.Cu) (net 31))
   (segment (start 162.56 73.787) (end 162.84 74.067) (width 0.3556) (layer B.Cu) (net 31))
