File: tempcontroll/tempcontroll.kicad_pcb (KiCad board)
At the start: 2 copper layers, 80 x 80 mm, 48 parts, among them J1 REL1, J10 REL2B, J11 Conn_01x03, J12 AVR_SPI, J2 -5V, J3 +24V, J4 +5V, J5 GND, J6 +D, J7 -TS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

Commit message: Prefinal work with pcb
Parts:
- added C1: 47u, Capacitors_Tantalum_SMD:CP_Tantalum_Case-D_EIA-7343-31_Reflow, B.Cu at (113.0, 106.7)
- added C10: 47u, Capacitors_Tantalum_SMD:CP_Tantalum_Case-D_EIA-7343-31_Reflow, B.Cu at (118.7, 59.7)
- added C11: 47u, Capacitors_Tantalum_SMD:CP_Tantalum_Case-D_EIA-7343-31_Reflow, B.Cu at (110.5, 55.2)
- added C12: 100n, Capacitors_SMD:C_0805, B.Cu at (159.0, 69.8)
- added C3: 1u, Capacitors_Tantalum_SMD:CP_Tantalum_Case-T_EIA-3528-12_Reflow, B.Cu at (152.4, 99.3)
- added C9: 47u, Capacitors_Tantalum_SMD:CP_Tantalum_Case-D_EIA-7343-31_Reflow, B.Cu at (144.8, 109.9)
- added Q4: BC807, TO_SOT_Packages_SMD:SOT-23, B.Cu at (105.6, 60.2)
- added Q5: BC807, TO_SOT_Packages_SMD:SOT-23, B.Cu at (175.3, 69.6)
- added R21: 1k, Resistors_SMD:R_0805, B.Cu at (129.5, 116.5)
- added R22: 1k, Resistors_SMD:R_0805, B.Cu at (165.5, 58.4)
- added SW1: Rotary_Encoder, MY:ENC1, F.Cu at (140.0, 90.0)
- C8: value 100u -> 100n
- moved R12 44.2 mm to (166.6, 53.3), turned to 0 degrees
- moved R4 28.4 mm to (124.2, 103.8), turned to 270 degrees
- moved C5 27.4 mm to (112.8, 77.5)
- moved R11 25.8 mm to (162.6, 103.2), turned to 270 degrees
- moved C2 19.8 mm to (131.2, 113.0)
- moved J11 19.2 mm to (135.9, 113.0)
- moved U1 19.2 mm to (127.0, 113.0)
- moved J12 17.8 mm to (114.3, 83.8), turned to 180 degrees
- moved R1 16.9 mm to (116.8, 93.7), turned to 270 degrees
- moved D1 15.7 mm to (113.0, 99.1)
- moved C7 15.2 mm to (166.1, 99.1)
- moved R16 15.2 mm to (167.6, 91.4)
- moved R14 11.6 mm to (163.5, 91.4), turned to 180 degrees
- moved C6 10.4 mm to (123.2, 97.8), turned to 0 degrees
- moved R7 8.31 mm to (138.8, 54.0), turned to 180 degrees
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Connections:
- net Net-(D3-Pad1) renamed /IN
- J3 pad 1: Net-(J3-Pad1) -> /+24V
- U1 pad 11: Net-(U1-Pad11) -> /REL2_O
- U1 pad 13: /LED -> Net-(SW1-Pad3)
- U1 pad 26: /D3 -> /D1
- U1 pad 28: /D1 -> /D3
- U1 pad 5: Net-(U1-Pad5) -> /LED
- U1 pad 6: Net-(U1-Pad6) -> /REL1_O
Routing:
- net Net-(Q4-Pad1): track 0.00 -> 106.6 mm
- net +5V: track 349.6 -> 253.1 mm, vias 2 -> 0
- net GND: track 211.6 -> 303.8 mm
- net /+24V: track 0.00 -> 83.6 mm, vias 0 -> 2
- net /LED: track 43.6 -> 113.9 mm
- net /REL2_O: track 0.00 -> 56.1 mm
- net Net-(D2-Pad2): track 57.2 -> 6.64 mm
- net Net-(Q5-Pad1): track 0.00 -> 48.3 mm
- net Net-(R11-Pad2): track 17.7 -> 64.3 mm
- net Net-(C3-Pad1): track 37.2 -> 12.5 mm
- net /REL1_O: track 0.00 -> 23.9 mm
- net Net-(R7-Pad2): track 20.4 -> 40.2 mm
- net /MOSI: track 31.1 -> 50.5 mm
- net Net-(D3-Pad2): track 36.8 -> 18.3 mm
- net Net-(SW1-Pad1): track 0.00 -> 17.9 mm
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Other:
- net class Default: via_dia 2 -> 2.3
- net class Power: via_dia 2 -> 2.3

Commit message: Final pcb
Parts:
- Q4, Q5: value BC807 -> 2SD667; footprint TO_SOT_Packages_SMD:SOT-23 -> TO_SOT_Packages_THT:TO-92_Molded_Narrow; moved to F.Cu
- R21, R22: value 1k -> 4k7
- moved Q5 67.3 mm to (108.0, 69.8), turned to 270 degrees
- moved Q4 65.9 mm to (171.4, 59.7), turned to 90 degrees
- moved R12 5.62 mm to (164.2, 48.3)
Connections:
- net Net-(C1-Pad1) renamed /AREF
- J3 pad 1: /+24V -> Net-(J3-Pad1)
- Q4 pad 1: Net-(Q4-Pad1) -> GND
- Q4 pad 2: /+24V -> Net-(J10-Pad1)
- Q4 pad 3: Net-(J1-Pad1) -> Net-(Q4-Pad3)
- Q5 pad 1: Net-(Q5-Pad1) -> GND
- Q5 pad 2: /+24V -> Net-(J1-Pad1)
- Q5 pad 3: Net-(J10-Pad1) -> Net-(Q5-Pad3)
- R21 pad 2: Net-(Q4-Pad1) -> Net-(Q5-Pad3)
- R22 pad 2: Net-(Q5-Pad1) -> Net-(Q4-Pad3)
Routing:
- net Net-(Q4-Pad1): track 106.6 -> 0.00 mm
- net Net-(Q5-Pad3): track 0.00 -> 89.1 mm
- net /+24V: track 83.6 -> 0.00 mm, vias 2 -> 0
- net Net-(Q5-Pad1): track 48.3 -> 0.00 mm
- net GND: track 303.8 -> 343.0 mm
- net +5V: track 253.1 -> 269.4 mm
- net Net-(Q4-Pad3): track 0.00 -> 7.46 mm
- net /D3: track 102.4 -> 106.6 mm
- net /D2: track 109.3 -> 113.5 mm
- net /D1: track 106.7 -> 111.0 mm
- net Net-(J10-Pad1): track 5.33 -> 9.16 mm
- net -5V: track 79.7 -> 76.8 mm
- net Net-(J1-Pad1): track 4.40 -> 7.04 mm
- net Net-(D2-Pad2): track 6.64 -> 4.50 mm
- net /LED: track 113.9 -> 112.9 mm

Commit message: Output pcb
Parts:
- moved SW1 1.00 mm to (140.0, 91.0)
Routing:
- net GND: track 343.0 -> 344.0 mm
- net Net-(SW1-Pad1): track 17.9 -> 17.1 mm
- net Net-(Q4-Pad3): track 7.46 -> 6.84 mm
Other:
- net class Default: clearance 0.2 -> 0.1
- rule trace_clearance: 0.2 -> 0.1
- board text added: "+24V"
- board text added: "+5V"
- board text added: "+TS"
- board text added: "-5V"
- board text added: "BOTTOM"
- board text added: "GND"
- board text added: "REL1"
- board text added: "REL2"

Commit message: Solder pcb
Other:
- net class Default: clearance 0.1 -> 0.11
- rule trace_clearance: 0.1 -> 0.11
Changed lines of the file:
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@@
     (user_trace_width 0.6)
     (user_trace_width 0.7)
-    (trace_clearance 0.1)
+    (trace_clearance 0.11)
     (zone_clearance 0.508)
     (zone_45_only no)
@@
   (net 57 "Net-(J3-Pad1)")
   (net_class Default "This is the default net class."
-    (clearance 0.1)
+    (clearance 0.11)
     (trace_width 0.3556)
     (via_dia 2.3)
@@
   (segment (start 112 68.213) (end 112.666213 68.879213) (width 0.4) (layer B.Cu) (net 32))
   (segment (start 112.666213 68.879213) (end 112.666213 71.12) (width 0.4) (layer B.Cu) (net 32))
+  (segment (start 162.56 68.58) (end 163 68.14) (width 0.4) (layer B.Cu) (net 35))
+  (segment (start 163 68.14) (end 163 65) (width 0.4) (layer B.Cu) (net 35))
+  (segment (start 162.56 69.85) (end 162.56 68.58) (width 0.4) (layer B.Cu) (net 35))
+  (segment (start 162.56 69.85) (end 160.004 69.85) (width 0.4) (layer B.Cu) (net 35))
   (segment (start 172.593 58.42) (end 173 58.827) (width 0.4) (layer B.Cu) (net 38))
   (segment (start 173 58.827) (end 173 65) (width 0.4) (layer B.Cu) (net 38))
@@
   (segment (start 164.597 58.42) (end 162.687 58.42) (width 0.4) (layer B.Cu) (net 51))
   (segment (start 125.603 81.394002) (end 125.603 87.63) (width 0.4) (layer B.Cu) (net 51))
+  (segment (start 162.56 73.34) (end 162.56 74.0456) (width 0.3556) (layer B.Cu) (net 53) (status 1000000))
+  (segment (start 162.56 74.0456) (end 162.56 77.47) (width 0.3556) (layer B.Cu) (net 53) (status 1000000))
+  (segment (start 162.56 77.47) (end 162.56 79.1756) (width 0.3556) (layer B.Cu) (net 53) (status 1000000))
+  (segment (start 162.56 79.1756) (end 162.56 82.55) (width 0.3556) (layer B.Cu) (net 53) (status 1000000))
+  (segment (start 162.56 82.55) (end 162.56 84.2556) (width 0.3556) (layer B.Cu) (net 53) (status 1000000))
+  (segment (start 162.56 84.2556) (end 162.56 87.63) (width 0.3556) (layer B.Cu) (net 53) (status 1000000))
   (segment (start 113.03 99.06) (end 113.03 103.505) (width 0.4) (layer B.Cu) (net 54))
   (segment (start 116.84 94.61) (end 118.74 94.61) (width 0.4) (layer B.Cu) (net 54))
@@
   (via (at 112.666213 71.12) (size 2.3) (drill 0.4) (layers F.Cu B.Cu) (net 32))
   (segment (start 112 65) (end 112 68.213) (width 0.4) (layer B.Cu) (net 32))
-  (segment (start 162.56 69.85) (end 160.004 69.85) (width 0.4) (layer B.Cu) (net 35))
-  (segment (start 162.56 69.85) (end 162.56 68.58) (width 0.4) (layer B.Cu) (net 35))
   (segment (start 162.56 71.44) (end 162.56 69.85) (width 0.4) (layer B.Cu) (net 35))
   (segment (start 165.42 69.85) (end 164.67 69.85) (width 0.4) (layer B.Cu) (net 35))
   (segment (start 164.67 69.85) (end 162.56 69.85) (width 0.4) (layer B.Cu) (net 35))
-  (segment (start 162.56 68.58) (end 163 68.14) (width 0.4) (layer B.Cu) (net 35))
-  (segment (start 163 68.14) (end 163 65) (width 0.4) (layer B.Cu) (net 35))
   (segment (start 138.049 115.443) (end 150.207 115.443) (width 0.4) (layer B.Cu) (net 36))
   (segment (start 120.938989 101.888989) (end 120.938989 106.714989) (width 0.4) (layer B.Cu) (net 36))
@@
   (segment (start 127.254 76.962) (end 141.036 63.18) (width 0.4) (layer B.Cu) (net 37))
   (segment (start 141.036 63.18) (end 143.51 63.18) (width 0.4) (layer B.Cu) (net 37))
-  (segment (start 162.56 73.34) (end 162.56 74.0456) (width 0.3556) (layer B.Cu) (net 53))
-  (segment (start 162.56 74.0456) (end 162.56 77.47) (width 0.3556) (layer B.Cu) (net 53))
   (segment (start 129 52) (end 127.34 53.66) (width 0.4) (layer B.Cu) (net 42))
   (segment (start 127.34 53.66) (end 125.19 53.66) (width 0.4) (layer B.Cu) (net 42))
@@
   (segment (start 125.603 105.537) (end 125.603 100.33) (width 0.4) (layer B.Cu) (net 52))
   (segment (start 125.603 100.33) (end 127 100.33) (width 0.4) (layer B.Cu) (net 52))
-  (segment (start 162.56 82.55) (end 162.56 84.2556) (width 0.3556) (layer B.Cu) (net 53))
-  (segment (start 162.56 84.2556) (end 162.56 87.63) (width 0.3556) (layer B.Cu) (net 53))
-  (segment (start 162.56 77.47) (end 162.56 79.1756) (width 0.3556) (layer B.Cu) (net 53))
-  (segment (start 162.56 79.1756) (end 162.56 82.55) (width 0.3556) (layer B.Cu) (net 53))
   (segment (start 107.315 84.328) (end 109.474 82.169) (width 0.4) (layer B.Cu) (net 55))
   (segment (start 117.602 110.871) (end 116.205 112.268) (width 0.4) (layer B.Cu) (net 55))
