File: tempcontroll/tempcontroll.sch (KiCad schematic (older format))
At the start: 30 parts, among them J1 AVR_SPI, J2 Conn_01x03, SW1 Rotary_Encoder_Switch, U1 ATMEGA8-16AU, U2 KL-4031-BSR, U3 OP07

Commit message: Start work
Parts:
- removed U1: ATMEGA8-16AU, Housings_QFP:LQFP-32_7x7mm_Pitch0.8mm, symbol atmel:ATMEGA8-16AU
- added C4, C5, C6, C7, C8: 100u, Capacitors_SMD:C_0805, symbol device:C
- added J1: REL1, MY:PAD, symbol Connector:Conn_01x01
- added J10: REL2B, MY:PAD, symbol Connector:Conn_01x01
- added J2: -5V, MY:PAD, symbol Connector:Conn_01x01
- added J3: +24V, MY:PAD, symbol Connector:Conn_01x01
- added J4: +5V, MY:PAD, symbol Connector:Conn_01x01
- added J5: GND, MY:PAD, symbol Connector:Conn_01x01
- added J6: +D, MY:PAD, symbol Connector:Conn_01x01
- added J7: -TS, MY:PAD, symbol Connector:Conn_01x01
- added J8: +TS, MY:PAD, symbol Connector:Conn_01x01
- added J9: REL2A, MY:PAD, symbol Connector:Conn_01x01
- added Q1, Q2, Q3: BC807, TO_SOT_Packages_SMD:SOT-23, symbol Transistor:BC807
- added R18, R19, R20: 1k, Resistors_SMD:R_0805, symbol device:R
- added U1: ATMEGA8-16PU, Housings_DIP:DIP-28_W7.62mm, symbol atmel:ATMEGA8-16PU
- renumbered J2 to J11, J1 to J12, R12 to R11, R11 to R12, R3 to R2, R4 to R3, R2 to R4
Connections:
- net labels added: TS
- wire segments 115 -> 161
- no-connect marks 10 -> 7

Commit message: Start coding 2
Changed lines of the file:
@@
 	6400 3900 6600 3900
 Text Label 6600 4100 0    60   ~ 0
-D1
+D3
 Text Label 6600 4000 0    60   ~ 0
 D2
 Text Label 6600 3900 0    60   ~ 0
-D3
+D1
 NoConn ~ 6400 3800
 NoConn ~ 6400 3700

Commit message: Prefinal work with pcb
Parts:
- removed SW1: Rotary_Encoder_Switch, symbol device:Rotary_Encoder_Switch
- added C10, C11, C9: 47u, Capacitors_Tantalum_SMD:CP_Tantalum_Case-D_EIA-7343-31_Reflow, symbol device:CP
- added C12: 100n, Capacitors_SMD:C_0805, symbol device:C
- added Q4, Q5: BC807, TO_SOT_Packages_SMD:SOT-23, symbol Transistor:BC807
- added R21, R22: 1k, Resistors_SMD:R_0805, symbol device:R
- added SW1: Rotary_Encoder, MY:ENC1, symbol device:Rotary_Encoder
- C1: footprint (none) -> Capacitors_Tantalum_SMD:CP_Tantalum_Case-D_EIA-7343-31_Reflow
- C3: footprint (none) -> Capacitors_Tantalum_SMD:CP_Tantalum_Case-T_EIA-3528-12_Reflow
- C8: value 100u -> 100n
Connections:
- net labels added: +24V, IN, REL1_O, REL2_O
- wire segments 161 -> 185

Commit message: Final pcb
Parts:
- removed Q4, Q5: BC807, TO_SOT_Packages_SMD:SOT-23, symbol Transistor:BC807
- added Q? (x2): 2SD667, TO_SOT_Packages_THT:TO-92_Molded_Narrow, symbol device:Q_NPN_ECB
- R21, R22: value 1k -> 4k7
Connections:
- net labels added: AREF
- net labels removed: +24V
- wire segments 185 -> 181
Changed lines of the file:
@@
 	0    1    1    0
 $EndComp
-Wire Wire Line
-	3450 3200 3500 3200
 $Comp
 L power:GND #PWR04
@@
 	3650 2600 3650 3100
 Wire Wire Line
-	3500 2950 3500 3200
-Connection ~ 3500 3200
-Wire Wire Line
-	3500 3200 4500 3200
-Wire Wire Line
 	3400 3500 3500 3500
 Wire Wire Line
@@
 Wire Wire Line
 	3300 3350 3500 3350
-Connection ~ 3500 3350
-Wire Wire Line
-	3500 3350 3500 3200
 $Comp
 L power:GND #PWR05
@@
 Connection ~ 10350 3300
 $Comp
-L Transistor:BC807 Q4
-U 1 1 5A3DCDF6
-P 2250 2350
-F 0 "Q4" H 2100 2250 50  0000 L CNN
-F 1 "BC807" H 1950 2150 50  0000 L CNN
-F 2 "TO_SOT_Packages_SMD:SOT-23" H 2450 2275 50  0001 L CIN
-F 3 "http://www.fairchildsemi.com/ds/BC/BC807.pdf" H 2250 2350 50  0001 L CNN
-	1    2250 2350
-	-1   0    0    -1
-$EndComp
-Wire Wire Line
-	1550 2100 2150 2100
-Wire Wire Line
-	2150 2100 2150 2150
-Wire Wire Line
-	1550 2500 1700 2500
-Wire Wire Line
-	1700 2500 1700 2600
-Wire Wire Line
-	1700 2600 2150 2600
-Wire Wire Line
-	2150 2600 2150 2550
-$Comp
 L device:R R21
 U 1 1 5A3EE566
 P 2700 2350
 F 0 "R21" V 2493 2350 50  0000 C CNN
-F 1 "1k" V 2584 2350 50  0000 C CNN
+F 1 "4k7" V 2584 2350 50  0000 C CNN
 F 2 "Resistors_SMD:R_0805" V 2630 2350 50  0001 C CNN
 F 3 "" H 2700 2350 50  0001 C CNN
@@
 	0    1    1    0
 $EndComp
-Wire Wire Line
-	2550 2350 2450 2350
 Wire Wire Line
 	2850 2350 2950 2350
@@
 NoConn ~ 1550 3700
 $Comp
-L Transistor:BC807 Q5
-U 1 1 5A441ACF
-P 2250 3600
-F 0 "Q5" H 2100 3500 50  0000 L CNN
-F 1 "BC807" H 1950 3400 50  0000 L CNN
-F 2 "TO_SOT_Packages_SMD:SOT-23" H 2450 3525 50  0001 L CIN
-F 3 "http://www.fairchildsemi.com/ds/BC/BC807.pdf" H 2250 3600 50  0001 L CNN
-	1    2250 3600
-	-1   0    0    1
-$EndComp
-Wire Wire Line
-	2150 3400 2150 2600
-Connection ~ 2150 2600
-Wire Wire Line
-	2150 3900 2150 3800
-$Comp
 L device:R R22
 U 1 1 5A454741
-P 2600 3900
-F 0 "R22" H 2530 3854 50  0000 R CNN
-F 1 "1k" H 2530 3945 50  0000 R CNN
-F 2 "Resistors_SMD:R_0805" V 2530 3900 50  0001 C CNN
-F 3 "" H 2600 3900 50  0001 C CNN
-	1    2600 3900
-	-1   0    0    1
-$EndComp
-Wire Wire Line
-	2600 3600 2600 3750
-Wire Wire Line
-	2450 3600 2600 3600
-Wire Wire Line
-	2600 4050 2600 4250
-Text Label 2600 4250 0    60   ~ 0
+P 2400 4200
+F 0 "R22" V 2300 4250 50  0000 R CNN
+F 1 "4k7" V 2500 4250 50  0000 R CNN
+F 2 "Resistors_SMD:R_0805" V 2330 4200 50  0001 C CNN
+F 3 "" H 2400 4200 50  0001 C CNN
+	1    2400 4200
+	0    1    1    0
+$EndComp
+Wire Wire Line
+	2550 4200 2950 4200
+Text Label 2950 4200 2    60   ~ 0
 REL2_O
-Wire Wire Line
-	1550 3900 2150 3900
-Text Label 1800 2600 0    60   ~ 0
-+24V
+Text Label 3800 3200 0    50   ~ 0
+AREF
+Connection ~ 3500 3350
+Wire Wire Line
+	3500 3350 3500 3200
+Wire Wire Line
+	3500 3200 4500 3200
+Connection ~ 3500 3200
+Wire Wire Line
+	3500 2950 3500 3200
+Wire Wire Line
+	3450 3200 3500 3200
+$Comp
+L device:Q_NPN_ECB Q?
+U 1 1 5A409982
+P 2250 2350
+F 0 "Q?" H 2100 2450 50  0000 L CNN
+F 1 "2SD667" H 1950 2200 50  0000 L CNN
+F 2 "TO_SOT_Packages_THT:TO-92_Molded_Narrow" H 2450 2450 50  0001 C CNN
+F 3 "" H 2250 2350 50  0001 C CNN
+	1    2250 2350
+	-1   0    0    -1
+$EndComp
+Wire Wire Line
+	1550 2100 2150 2100
+Wire Wire Line
+	2150 2100 2150 2150
+$Comp
+L power:GND #PWR?
+U 1 1 5A412B11
+P 2150 2650
+F 0 "#PWR?" H 2150 2400 50  0001 C CNN
+F 1 "GND" H 2155 2477 50  0000 C CNN
+F 2 "" H 2150 2650 50  0001 C CNN
+F 3 "" H 2150 2650 50  0001 C CNN
+	1    2150 2650
+	1    0    0    -1
+$EndComp
+Wire Wire Line
+	2150 2650 2150 2550
+Wire Wire Line
+	2450 2350 2550 2350
+$Comp
+L device:Q_NPN_ECB Q?
+U 1 1 5A424860
+P 1900 4200
+F 0 "Q?" H 1750 4300 50  0000 L CNN
+F 1 "2SD667" H 1600 4050 50  0000 L CNN
+F 2 "TO_SOT_Packages_THT:TO-92_Molded_Narrow" H 2100 4300 50  0001 C CNN
+F 3 "" H 1900 4200 50  0001 C CNN
+	1    1900 4200
+	-1   0    0    -1
+$EndComp
+Wire Wire Line
+	1550 3900 1800 3900
+Wire Wire Line
+	1800 3900 1800 4000
+$Comp
+L power:GND #PWR?
+U 1 1 5A42DD0E
+P 1800 4500
+F 0 "#PWR?" H 1800 4250 50  0001 C CNN
+F 1 "GND" H 1805 4327 50  0000 C CNN
+F 2 "" H 1800 4500 50  0001 C CNN
+F 3 "" H 1800 4500 50  0001 C CNN
+	1    1800 4500
+	1    0    0    -1
+$EndComp
+Wire Wire Line
+	1800 4400 1800 4500
+Wire Wire Line
+	2250 4200 2100 4200
 $EndSCHEMATC

Commit message: Solder pcb
Parts:
- R12: value 330 -> 470
- gave numbers to parts that had none: 2
Changed lines of the file:
@@
 P 7700 4600
 F 0 "R12" V 7650 4400 50  0000 C CNN
-F 1 "330" V 7700 4600 50  0000 C CNN
+F 1 "470" V 7700 4600 50  0000 C CNN
 F 2 "Resistors_SMD:R_0805" V 7630 4600 50  0001 C CNN
 F 3 "" H 7700 4600 50  0001 C CNN
@@
 	3450 3200 3500 3200
 $Comp
-L device:Q_NPN_ECB Q?
+L device:Q_NPN_ECB Q5
 U 1 1 5A409982
 P 2250 2350
-F 0 "Q?" H 2100 2450 50  0000 L CNN
+F 0 "Q5" H 2100 2450 50  0000 L CNN
 F 1 "2SD667" H 1950 2200 50  0000 L CNN
 F 2 "TO_SOT_Packages_THT:TO-92_Molded_Narrow" H 2450 2450 50  0001 C CNN
@@
 	2150 2100 2150 2150
 $Comp
-L power:GND #PWR?
+L power:GND #PWR023
 U 1 1 5A412B11
 P 2150 2650
-F 0 "#PWR?" H 2150 2400 50  0001 C CNN
+F 0 "#PWR023" H 2150 2400 50  0001 C CNN
 F 1 "GND" H 2155 2477 50  0000 C CNN
 F 2 "" H 2150 2650 50  0001 C CNN
@@
 	2450 2350 2550 2350
 $Comp
-L device:Q_NPN_ECB Q?
+L device:Q_NPN_ECB Q4
 U 1 1 5A424860
 P 1900 4200
-F 0 "Q?" H 1750 4300 50  0000 L CNN
+F 0 "Q4" H 1750 4300 50  0000 L CNN
 F 1 "2SD667" H 1600 4050 50  0000 L CNN
 F 2 "TO_SOT_Packages_THT:TO-92_Molded_Narrow" H 2100 4300 50  0001 C CNN
@@
 	1800 3900 1800 4000
 $Comp
-L power:GND #PWR?
+L power:GND #PWR032
 U 1 1 5A42DD0E
 P 1800 4500
-F 0 "#PWR?" H 1800 4250 50  0001 C CNN
+F 0 "#PWR032" H 1800 4250 50  0001 C CNN
 F 1 "GND" H 1805 4327 50  0000 C CNN
 F 2 "" H 1800 4500 50  0001 C CNN

Commit message: Start write soft
Parts:
- R10, R2, R3, R5, R6, R7, R8, R9: value 220 -> 470
Changed lines of the file:
@@
 P 7150 2900
 F 0 "R5" V 7100 2700 50  0000 C CNN
-F 1 "220" V 7150 2900 50  0000 C CNN
+F 1 "470" V 7150 2900 50  0000 C CNN
 F 2 "Resistors_SMD:R_0805" V 7080 2900 50  0001 C CNN
 F 3 "" H 7150 2900 50  0001 C CNN
@@
 P 7150 3000
 F 0 "R6" V 7100 2800 50  0000 C CNN
-F 1 "220" V 7150 3000 50  0000 C CNN
+F 1 "470" V 7150 3000 50  0000 C CNN
 F 2 "Resistors_SMD:R_0805" V 7080 3000 50  0001 C CNN
 F 3 "" H 7150 3000 50  0001 C CNN
@@
 P 7150 3100
 F 0 "R7" V 7100 2900 50  0000 C CNN
-F 1 "220" V 7150 3100 50  0000 C CNN
+F 1 "470" V 7150 3100 50  0000 C CNN
 F 2 "Resistors_SMD:R_0805" V 7080 3100 50  0001 C CNN
 F 3 "" H 7150 3100 50  0001 C CNN
@@
 P 7150 3200
 F 0 "R8" V 7100 3000 50  0000 C CNN
-F 1 "220" V 7150 3200 50  0000 C CNN
+F 1 "470" V 7150 3200 50  0000 C CNN
 F 2 "Resistors_SMD:R_0805" V 7080 3200 50  0001 C CNN
 F 3 "" H 7150 3200 50  0001 C CNN
@@
 P 7150 3300
 F 0 "R9" V 7100 3100 50  0000 C CNN
-F 1 "220" V 7150 3300 50  0000 C CNN
+F 1 "470" V 7150 3300 50  0000 C CNN
 F 2 "Resistors_SMD:R_0805" V 7080 3300 50  0001 C CNN
 F 3 "" H 7150 3300 50  0001 C CNN
@@
 P 7150 3400
 F 0 "R10" V 7100 3200 50  0000 C CNN
-F 1 "220" V 7150 3400 50  0000 C CNN
+F 1 "470" V 7150 3400 50  0000 C CNN
 F 2 "Resistors_SMD:R_0805" V 7080 3400 50  0001 C CNN
 F 3 "" H 7150 3400 50  0001 C CNN
@@
 P 4150 3600
 F 0 "R2" V 4050 3600 50  0000 C CNN
-F 1 "220" V 4150 3600 50  0000 C CNN
+F 1 "470" V 4150 3600 50  0000 C CNN
 F 2 "Resistors_SMD:R_0805" V 4080 3600 50  0001 C CNN
 F 3 "" H 4150 3600 50  0001 C CNN
@@
 P 4150 3800
 F 0 "R3" V 4050 3800 50  0000 C CNN
-F 1 "220" V 4150 3800 50  0000 C CNN
+F 1 "470" V 4150 3800 50  0000 C CNN
 F 2 "Resistors_SMD:R_0805" V 4080 3800 50  0001 C CNN
 F 3 "" H 4150 3800 50  0001 C CNN
